File: baksteen-opl2/hardware/hardware.kicad_pcb (KiCad board)
At the start: 2 copper layers, 48.8 x 105 mm, 48 parts, among them J1 AudioJack2, J10 Eurorack Power, J11 OPL, J2 AudioJack2, J3 AudioJack2, J4 AudioJack2, J5 AudioJack2, J6 AudioJack2, J7 AudioJack2, J8 AudioJack2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

Commit message: removed nano, going with bare atmega328p in tqfp package
Parts:
- removed A1: Nano v3.x, Module:Arduino_Nano_WithMountingHoles
- added C4: 100nF, Capacitor_SMD:C_0805_2012Metric, B.Cu at (206.1, 50.0)
- added C5: 22pF, Capacitor_SMD:C_0805_2012Metric, B.Cu at (200.1, 60.0)
- added C6: 22pF, Capacitor_SMD:C_0805_2012Metric, B.Cu at (200.1, 55.0)
- added C7: 100nF, Capacitor_SMD:C_0805_2012Metric, B.Cu at (200.1, 50.0)
- added J12: OPL, Connector_PinSocket_2.54mm:PinSocket_1x07_P2.54mm_Vertical, B.Cu at (229.0, 72.4)
- added R15: 10k, Resistor_SMD:R_0805_2012Metric, B.Cu at (206.1, 55.0)
- added U3: LM7805_TO220, Package_TO_SOT_SMD:SOT-223-3_TabPin2, B.Cu at (188.0, 96.0)
- added Y1: 16Mhz, Crystal:Crystal_HC52-6mm_Vertical, B.Cu at (214.0, 52.0)
- J11: value OPL -> ICSP; footprint Connector_PinSocket_2.54mm:PinSocket_1x07_P2.54mm_Vertical -> Connector_IDC:IDC-Header_2x03_P2.54mm_Vertical
- R1, R2, R3: value 10k -> 100k
- R10, R11, R9: value 100k -> 10k
- R12, R13, R14: value 100 -> 10k
- R4, R5, R6: value 10k -> 100
- U2: value LM7805_TO220 -> ATmega328PB-A; footprint Package_TO_SOT_SMD:SOT-223-3_TabPin2 -> Package_QFP:TQFP-32_7x7mm_P0.8mm
- moved U2 56.0 mm to (225.0, 54.0), turned to 90 degrees
- moved J11 51.9 mm to (228.5, 28.5)
Connections:
- C1 pad 1: CV2 -> V/OCT
- C2 pad 1: CV2 -> CV1
- D10 pad 1: CV2 -> V/OCT
- D11 pad 2: CV2 -> CV1
- D12 pad 1: CV2 -> CV1
- D9 pad 2: CV2 -> V/OCT
- J1 pad T: GATE1 -> Net-(J1-PadT)
- J11 pad 1: 5V -> MISO
- J11 pad 2: GND -> 5V
- J11 pad 3: A0 -> OPL_SHIFT
- J11 pad 4: DATA -> MOSI
- J11 pad 5: LATCH -> RESET
- J11 pad 6: SHIFT -> GND
- J2 pad T: GATE2 -> Net-(J2-PadT)
- J3 pad T: GATE3 -> Net-(J3-PadT)
- J4 pad T: GATE4 -> GATE1
- J5 pad T: GATE5 -> GATE2
- J6 pad T: GATE6 -> GATE3
- J7 pad T: Net-(J7-PadT) -> GATE4
- J8 pad T: Net-(J8-PadT) -> GATE5
- J9 pad T: Net-(J9-PadT) -> GATE6
- R1 pad 1: GND -> Net-(J1-PadT)
- R1 pad 2: Next -> GND
- R10 pad 1: Net-(J8-PadT) -> GND
- R10 pad 2: GND -> GATE2
- R11 pad 1: Net-(J9-PadT) -> GND
- R11 pad 2: GND -> GATE3
- R12 pad 1: Net-(J7-PadT) -> GND
- R12 pad 2: CV2 -> GATE4
- R13 pad 1: Net-(J8-PadT) -> GND
- R13 pad 2: CV2 -> GATE5
- R14 pad 1: Net-(J9-PadT) -> GND
- R14 pad 2: CV2 -> GATE6
- R2 pad 1: GND -> Net-(J2-PadT)
- R2 pad 2: Prev -> GND
- R3 pad 1: GND -> Net-(J3-PadT)
- R3 pad 2: GATE1 -> GND
- R4 pad 1: GND -> Net-(J1-PadT)
- R4 pad 2: GATE2 -> V/OCT
- R5 pad 1: GND -> Net-(J2-PadT)
- R5 pad 2: GATE3 -> CV1
- R6 pad 1: GND -> Net-(J3-PadT)
- R6 pad 2: GATE4 -> CV2
- R7 pad 2: GATE5 -> Next
- R8 pad 2: GATE6 -> Prev
- R9 pad 1: Net-(J7-PadT) -> GND
- R9 pad 2: GND -> GATE1
- U1 pad 7: SHIFT_DATAOUT -> MISO
- U2 pad 1: +12V -> ENC_2
- U2 pad 2: GND -> SHIFT_CLKIN
- U2 pad 3: 5V -> unconnected-(U2-Pad3)

Commit message: added tracks ... mostly
Parts:
- C5, C6, J12: moved to F.Cu
- J1: value AudioJack2 -> V/OCT
- J2: value AudioJack2 -> CV1
- J3: value AudioJack2 -> CV2
- J4: value AudioJack2 -> GATE1
- J5: value AudioJack2 -> GATE2
- J6: value AudioJack2 -> GATE3
- J7: value AudioJack2 -> GATE4
- J8: value AudioJack2 -> GATE5
- J9: value AudioJack2 -> GATE6
- moved R6 66.9 mm to (225.1, 124.0), turned to 0 degrees
- moved R5 57.2 mm to (213.0, 124.0), turned to 0 degrees
- moved R3 52.8 mm to (217.8, 124.0)
- moved R4 48.8 mm to (201.0, 124.0), turned to 0 degrees
- moved D8 46.1 mm to (221.0, 88.2)
- moved D7 45.5 mm to (209.6, 88.2)
- moved R2 43.3 mm to (206.0, 123.9)
- moved R11 42.3 mm to (224.2, 81.6)
- moved R10 42.2 mm to (213.0, 81.8)
- moved R9 42.2 mm to (201.0, 81.8)
- moved J1 41.6 mm to (197.2, 112.8)
- moved J2 41.6 mm to (209.2, 112.8)
- moved J3 41.6 mm to (221.0, 112.6)
- moved R1 35.7 mm to (194.0, 124.0)
- moved C6 32.6 mm to (229.0, 70.0), turned to -90 degrees
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Connections:
- J1 pad S: GND -> unconnected-(J1-PadS)
- J1 pad T: Net-(J1-PadT) -> GND
- J2 pad S: GND -> unconnected-(J2-PadS)
- J2 pad T: Net-(J2-PadT) -> GND
- J3 pad S: GND -> unconnected-(J3-PadS)
- J3 pad T: Net-(J3-PadT) -> GND
- R1 pad 1: Net-(J1-PadT) -> GND
- R2 pad 1: Net-(J2-PadT) -> GND
- R3 pad 1: Net-(J3-PadT) -> GND
- R4 pad 1: Net-(J1-PadT) -> GND
- R5 pad 1: Net-(J2-PadT) -> GND
- R6 pad 1: Net-(J3-PadT) -> GND
Routing:
- net 5V: track 0.00 -> 314.0 mm, vias 0 -> 8
- net MOSI: track 0.00 -> 126.3 mm
- net OPL_SHIFT: track 0.00 -> 105.8 mm, vias 0 -> 2
- net GATE6: track 0.00 -> 89.5 mm
- net MISO: track 0.00 -> 85.4 mm, vias 0 -> 1
- net GATE5: track 0.00 -> 77.4 mm
- net GATE3: track 0.00 -> 74.0 mm
- net GATE4: track 0.00 -> 69.9 mm
- net Next: track 0.00 -> 67.3 mm
- net GATE2: track 0.00 -> 64.4 mm
- net OPL_A0: track 0.00 -> 63.2 mm
- net OPL_LATCH: track 0.00 -> 61.2 mm, vias 0 -> 2
- net OPL_RESET: track 0.00 -> 58.4 mm, vias 0 -> 2
- net Net-(D5-Pad1): track 0.00 -> 54.6 mm
- net Prev: track 0.00 -> 52.3 mm
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- added copper zone on B.Cu, net GND
- added copper zone on F.Cu, net GND

Commit message: reran tracks ... mostly complete, couple DRC errors
Parts:
- J11: footprint Connector_IDC:IDC-Header_2x03_P2.54mm_Vertical -> Connector_PinHeader_2.54mm:PinHeader_2x03_P2.54mm_Vertical
- moved R7 38.8 mm to (215.2, 38.3), turned to 90 degrees
- moved R8 27.8 mm to (202.6, 38.2), turned to 90 degrees
- moved J11 23.5 mm to (229.9, 51.9)
- moved C6 14.7 mm to (223.4, 56.4), turned to 0 degrees
- moved R15 14.6 mm to (230.0, 64.6)
- moved Y1 14.4 mm to (219.0, 56.5)
- moved C7 10.6 mm to (230.0, 60.8), turned to 90 degrees
- moved C5 9.12 mm to (223.4, 52.8), turned to 0 degrees
- moved C4 8.16 mm to (227.4, 48.0)
- moved U2 1.84 mm to (208.6, 54.2), turned to 180 degrees
- moved U3 0.85 mm to (188.6, 96.6), turned to 180 degrees
- moved R2 0.29 mm to (206.0, 124.2)
- moved J10 0.22 mm to (187.4, 117.1)
- moved D8 0.20 mm to (221.0, 88.0), turned to -90 degrees
- moved R1 0.20 mm to (194.0, 124.2)
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Connections:
- J1 pad S: unconnected-(J1-PadS) -> GND
- J1 pad T: GND -> Net-(J1-PadT)
- J1 pad TN: (no net) -> unconnected-(J1-PadTN)
- J2 pad S: unconnected-(J2-PadS) -> GND
- J2 pad T: GND -> Net-(J2-PadT)
- J2 pad TN: (no net) -> unconnected-(J2-PadTN)
- J3 pad S: unconnected-(J3-PadS) -> GND
- J3 pad T: GND -> Net-(J3-PadT)
- J3 pad TN: (no net) -> unconnected-(J3-PadTN)
- J4 pad TN: (no net) -> unconnected-(J4-PadTN)
- J5 pad TN: (no net) -> unconnected-(J5-PadTN)
- J6 pad TN: (no net) -> unconnected-(J6-PadTN)
- J7 pad TN: (no net) -> unconnected-(J7-PadTN)
- J8 pad TN: (no net) -> unconnected-(J8-PadTN)
- J9 pad TN: (no net) -> unconnected-(J9-PadTN)
- R1 pad 1: GND -> Net-(J1-PadT)
- R2 pad 1: GND -> Net-(J2-PadT)
- R3 pad 1: GND -> Net-(J3-PadT)
- R4 pad 1: GND -> Net-(J1-PadT)
- R5 pad 1: GND -> Net-(J2-PadT)
- R6 pad 1: GND -> Net-(J3-PadT)
- U1 pad 10: NC -> unconnected-(U1-Pad10)
- U1 pad 9: NC -> unconnected-(U1-Pad9)
Routing:
- net 5V: track 314.0 -> 470.4 mm, vias 8 -> 4
- net CV2: track 0.00 -> 122.2 mm, vias 0 -> 2
- net CV1: track 0.00 -> 110.6 mm, vias 0 -> 2
- net V/OCT: track 0.00 -> 96.8 mm, vias 0 -> 2
- net MOSI: track 126.3 -> 74.5 mm, vias 0 -> 1
- net MISO: track 85.4 -> 50.7 mm, vias 1 -> 3
- net Net-(C6-Pad1): track 32.4 -> 9.85 mm, vias 1 -> 0
- net GATE2: track 64.4 -> 45.5 mm
- net Net-(C7-Pad1): track 19.3 -> 36.6 mm
- net Net-(C5-Pad1): track 29.2 -> 11.9 mm, vias 1 -> 0
- net RESET: track 19.7 -> 2.95 mm
- net OPL_A0: track 63.2 -> 46.5 mm
- net Net-(D1-Pad1): track 28.7 -> 13.4 mm
- net Next: track 67.3 -> 54.1 mm, vias 0 -> 1
- net OPL_SHIFT: track 105.8 -> 93.0 mm, vias 2 -> 1
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